File: mic_preamp_2ch.kicad_sch (KiCad schematic)
At the start: 47 parts, among them J1 NC3FAH1, J2 NC3FAH1, J3 PWR +15/GND/-15, J4 P48 +48/GND, J5 OUT1/GND/OUT2/GND, U1 INA163UA, U2 INA163UA

Commit message: v2: hand-routed symmetric input path, 0.1% matched parts, 10R series
Fixes the review of efc1e58: the 47R series resistors were a misreading of
datasheet Fig.2 (47R is in parallel with 1.2uH there) and doubled input noise.
Phantom feed is now 2x3.40k 0.1% per leg, bias 2.2k 0.1%, series 10R.
Input legs are routed by hand and locked; only power/phantom/GND autorouted.
Parts:
- added R10, R19, R20, R9: 3.40k, Resistor_SMD:R_1206_3216Metric, symbol Device:R
- R1, R11, R12, R2: value 6.81k -> 3.40k; footprint Resistor_SMD:R_2010_5025Metric -> Resistor_SMD:R_1206_3216Metric; LCSC C407009 -> C870711; MPN 201007F6811T4E -> RT1206BRD073K4L; Manufacturer UNI-ROYAL -> YAGEO; Spec 6.81k 1% 2010 0.75W 200V -> 3.40k 0.1% 25ppm thin film 1206 0.25W 200V; 2 in series per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
- R14, R15, R4, R5: LCSC C17520 -> C865371; MPN 0805W8F2201T5E -> RT0805BRD072K2L; Manufacturer UNI-ROYAL -> YAGEO; Spec 2.2k 1% 0805 -> 2.2k 0.1% 25ppm thin film 0805
- R16, R17, R6, R7: value 47R -> 10R; LCSC C17714 -> C55205321; MPN 0805W8F470JT5E -> CRF0805Q10R0BN; Manufacturer UNI-ROYAL -> SIE; Spec 47R 1% 0805 -> 10R 0.1% thin film 0805
Connections:
- net PH1: now also R10.1, R9.1; no longer R1.1, R2.1
- net PH2: now also R19.1, R20.1; no longer R11.1, R12.1
- new net P1C: R10.2, R2.1
- new net P1H: R1.1, R9.2
- new net P2C: R12.1, R20.2
- new net P2H: R11.1, R19.2
Other:
- note added: "D1/D2 BAV99 kep ve +/-15V (datasheet goi y 4x 1N4148). R6/R7 10R thin film: chia dong voi diode kep noi cua INA163 (abs max 10mA); nhieu them 0.57 nV/rtHz (2x10R) so voi 1 nV/rtHz cua IC."
- note added: "D21/D22 SMAJ16A: kep rail +/-15V khi cam/rut mic luc dang bat P48 (tu 47u nap 48V xa qua BAV99 vao rail). Khong co trong datasheet - them theo kinh nghiem thiet ke."
- note added: "Moi chan phantom = 2 x 3.40k 0.1% 1206 noi tiep (6.80k, khop 0.1% cho CMRR). Khi chan mic chap GND: 0.34W chia 2 = 0.17W/con (dinh muc 0.25W)."
- note added: "Ngo ra DC-coupled (khong lap servo OPA134 cua Fig.5): offset xau nhat ~0.25V o G=100 -> tang sau phai AC-couple."
- note removed: "D1/D2 BAV99 kep ve +/-15V (datasheet goi y 4x 1N4148). R6/R7 47R gioi han dong vao diode noi cua INA163 (abs max 10mA) - lay tu Fig.2."
- note removed: "D21/D22 SMAJ16A: kep rail +/-15V khi cam/rut mic luc dang bat P48 (tu 47u nap 48V xa qua BAV99 vao rail). Datasheet INA163 khong co phan nay - them theo kinh nghiem thiet ke."
- note removed: "R1/R2 6.81k 2010 (0.75W): khi chan mic chap GND, 48V roi het tren 1 dien tro = 0.34W."
